File: Hardware/RN41_Rootooth.brd (EAGLE design)
At the start: 41.1 x 22.6 mm, 23 parts, among them Q1 MOSFET-NCHANNELSMD, Q2 MOSFET-NCHANNELSMD, U1 V_REG_317SMD, U2 BLUETOOTH-RN41, U3 V_REG_LDOSMD

Commit message: Updated Revision to symbol layer
Parts:
- added U$2: REVISION, SparkFun-Aesthetics:REVISION
Other:
- board text added: "A. Weiss"
- board text added: "P. Lewis, T. Klopfenstein"
- board text removed: "A. Weiss, Revisions by: P. Lewis, T. Klopfenstein"
